File: exo_sequencer/exo_sequencer.sch (EAGLE design)
At the start: 111 parts, among them U1 THONKICONNNEW, U10 THONKICONNNEW, U11 THONKICONNNEW, U2 THONKICONNNEW, U3 THONKICONNNEW, U4 THONKICONNNEW, U5 THONKICONNNEW, U6 THONKICONNNEW, U7 THONKICONNNEW, U8 THONKICONNNEW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

Commit message: Add files via upload
Connections:
- net 3.3V: now also MCU.3.3V
Changed lines of the file:
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@@
 <part name="C1" library="SparkFun-Capacitors" deviceset="0.33UF/330NF" device="-0805-50V-10%" value="0.33µF"/>
 <part name="C2" library="SparkFun-Capacitors" deviceset="0.1UF" device="-0402-16V-10%" value="0.1uF"/>
+<part name="SUPPLY10" library="SparkFun-PowerSymbols" deviceset="3.3V" device=""/>
 </parts>
 <sheets>
@@
 <instance part="C1" gate="G$1" x="-58.42" y="2.54"/>
 <instance part="C2" gate="G$1" x="-17.78" y="5.08" rot="R180"/>
+<instance part="SUPPLY10" gate="G$1" x="-25.4" y="15.24"/>
 </instances>
 <busses>
@@
 <pinref part="SUPPLY9" gate="G$1" pin="3.3V"/>
 </segment>
-</net>
+<segment>
+<pinref part="MCU" gate="G$1" pin="3.3V"/>
+<wire x1="-5.08" y1="10.16" x2="-25.4" y2="10.16" width="0.1524" layer="91"/>
+<pinref part="SUPPLY10" gate="G$1" pin="3.3V"/>
+<wire x1="-25.4" y1="10.16" x2="-25.4" y2="15.24" width="0.1524" layer="91"/>
+</segment>
+</net>
